File: pocketcube_child_board/_autosave-pocketcube_child_board.kicad_pcb (KiCad board)
At the start: 2 copper layers, 50 x 50 mm, 4 parts, among them J1 M55-7102042R

Commit message: 11/2 via attempt
Routing:
- net GND: track 30.2 -> 38.9 mm, vias 0 -> 8
Changed lines of the file:
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@@
+	)
+	(segment
+		(start 121 57.5)
+		(end 122 57.5)
+		(width 0.2)
+		(layer "F.Cu")
+		(net 3)
 	)
 	(segment
@@
 	)
 	(segment
+		(start 116 57.5)
+		(end 117 57.5)
+		(width 0.2)
+		(layer "F.Cu")
+		(net 3)
+	)
+	(segment
 		(start 98.785 68)
 		(end 98.785 66.73)
@@
 	)
 	(segment
+		(start 115.5 57.5)
+		(end 116 57.5)
+		(width 0.2)
+		(layer "F.Cu")
+		(net 3)
+	)
+	(segment
+		(start 123 57.5)
+		(end 123.5 57.5)
+		(width 0.2)
+		(layer "F.Cu")
+		(net 3)
+	)
+	(segment
 		(start 92 46)
 		(end 92.5 45.5)
@@
 	)
 	(segment
+		(start 118 57.5)
+		(end 119 57.5)
+		(width 0.2)
+		(layer "F.Cu")
+		(net 3)
+	)
+	(segment
+		(start 117 57.5)
+		(end 118 57.5)
+		(width 0.2)
+		(layer "F.Cu")
+		(net 3)
+	)
+	(segment
 		(start 112 57.5)
 		(end 115.5 57.5)
 		(width 0.2)
 		(layer "F.Cu")
+		(net 3)
+	)
+	(segment
+		(start 119 57.5)
+		(end 120 57.5)
+		(width 0.2)
+		(layer "F.Cu")
+		(net 3)
+	)
+	(segment
+		(start 122 57.5)
+		(end 123 57.5)
+		(width 0.2)
+		(layer "F.Cu")
+		(net 3)
+	)
+	(segment
+		(start 123.5 57.5)
+		(end 124 58)
+		(width 0.2)
+		(layer "F.Cu")
+		(net 3)
+	)
+	(segment
+		(start 120 57.5)
+		(end 121 57.5)
+		(width 0.2)
+		(layer "F.Cu")
+		(net 3)
+	)
+	(via
+		(at 121 57.5)
+		(size 0.6)
+		(drill 0.3)
+		(layers "F.Cu" "B.Cu")
+		(net 3)
+	)
+	(via
+		(at 120 57.5)
+		(size 0.6)
+		(drill 0.3)
+		(layers "F.Cu" "B.Cu")
+		(net 3)
+	)
+	(via
+		(at 116 57.5)
+		(size 0.6)
+		(drill 0.3)
+		(layers "F.Cu" "B.Cu")
+		(net 3)
+	)
+	(via
+		(at 119 57.5)
+		(size 0.6)
+		(drill 0.3)
+		(layers "F.Cu" "B.Cu")
+		(net 3)
+	)
+	(via
+		(at 117 57.5)
+		(size 0.6)
+		(drill 0.3)
+		(layers "F.Cu" "B.Cu")
+		(net 3)
+	)
+	(via
+		(at 118 57.5)
+		(size 0.6)
+		(drill 0.3)
+		(layers "F.Cu" "B.Cu")
+		(net 3)
+	)
+	(via
+		(at 123 57.5)
+		(size 0.6)
+		(drill 0.3)
+		(layers "F.Cu" "B.Cu")
+		(net 3)
+	)
+	(via
+		(at 122 57.5)
+		(size 0.6)
+		(drill 0.3)
+		(layers "F.Cu" "B.Cu")
 		(net 3)
 	)
@@
 		(polygon
 			(pts
-				(xy 86.81797 43.31797) (xy 119.5 43.5) (xy 121 80.5) (xy 83 80) (xy 83.5 43.5)
+				(xy 86.81797 43.31797) (xy 123.500904 43.522284) (xy 125.002135 80.55266) (xy 83 80) (xy 83.5 43.5)
 			)
 		)
@@
 		(polygon
 			(pts
-				(xy 83.5 40.5) (xy 119.5 40) (xy 119.436867 77.724114) (xy 84.212772 77.591257) (xy 83.5 40)
+				(xy 83.5 40.5) (xy 118.493281 40.013982) (xy 118.430178 77.720317) (xy 84.212772 77.591257) (xy 83.5 40)
 			)
 		)
