File: pocketcube_child_board/pocketcube_child_board.kicad_pcb (KiCad board)
At the start: 4 copper layers, 47 x 47 mm, 17 parts, among them J1 M55-7102642R, J2 M55-7101242R, J3 M55-7101242R, J4 M55-7101242R, U1 SI3477DV-T1-GE3

Commit message: Pocketcube Monopole Antenna Board - Alex
Routing:
- net EXTERNAL_VOLTAGE: track 24.0 -> 79.9 mm, vias 0 -> 3
- net ANT_SPI2_MISO: track 0.00 -> 49.6 mm, vias 0 -> 3
- net /ANTENNA_TRACE: track 0.00 -> 48.6 mm, vias 0 -> 2
- net ANT_SPI2_MOSI: track 0.00 -> 47.5 mm, vias 0 -> 3
- net I2C3_SCL: track 0.00 -> 45.4 mm, vias 0 -> 2
- net I2C2_SDA: track 0.00 -> 38.7 mm, vias 0 -> 2
- net I2C3_SDA: track 0.00 -> 37.7 mm, vias 0 -> 2
- net I2C2_SCL: track 0.00 -> 36.2 mm, vias 0 -> 3
- net ANT_SPI2_SCK: track 0.00 -> 36.1 mm, vias 0 -> 3
- net ANT_SPI2_NSS: track 0.00 -> 32.3 mm, vias 0 -> 2
- net I2C1_SDA: track 0.00 -> 30.7 mm, vias 0 -> 2
- net I2C1_SCL: track 0.00 -> 28.5 mm, vias 0 -> 2
- net RFM_RESET: track 0.00 -> 20.4 mm, vias 0 -> 2
- net BAT_VOLTAGE: track 8.28 -> 27.6 mm
- net Net-(R_BURN1-Pad1): track 0.00 -> 10.5 mm
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