File: pocketcube_child_board/pocketcube_child_board.kicad_sch (KiCad schematic)
At the start: 7 parts, among them J1 M55-7102042R, U1 SI3477DV-T1-GE3

Commit message: PMOS Implementation and Ground Plane
Parts:
- renumbered R_BURN to R_BURN1, R_PULLUP to R_PULLUP1
Connections:
- net DIO0 is gone; now on net PMOS_GATE: R_PULLUP1.2, U1.3 (G)
- net PMOS_GATE: now also MOD1.7 (DIO5), MOD1.7_1 (DIO5__1); no longer MOD1.14 (DIO0), MOD1.14_1 (DIO0__1)
- net ANTENNA_TRACE: now reaches AE1.1 (A), MOD1.9 (ANT), MOD1.9_1 (ANT__1)

Commit message: Pushing Board sizes
Parts:
- removed J1: M55-7102042R, inspirefly:HARWIN_M55-7102042R, symbol inspireFly:M55-7102042R
- removed R_PULLUP1: 10k, symbol Device:R
- added C2, C3, C4, C5: 47uF, Capacitor_SMD:C_1206_3216Metric_Pad1.33x1.80mm_HandSolder, symbol Device:C
- added H1, H2, H3, H4: MountingHole_Pad, MountingHole:MountingHole_2.2mm_M2_Pad_TopBottom, symbol Mechanical:MountingHole_Pad
- added J1: M55-7102642R, inspirefly:HARWIN_M55-7102642R, symbol inspireFly:M55-7102642R
- added J2, J3, J4: M55-7101242R, inspirefly:HARWIN_M55-7101242R, symbol inspireFly:M55-7101242R
- added R1: 100K, Resistor_SMD:R_0402_1005Metric_Pad0.72x0.64mm_HandSolder, symbol Device:R_US
- MOD1: footprint inspirefly:RFM98W-433S2 -> inspirefly:XCVR_RFM98W-433S2
Connections:
- net GND: now also C2.1, C3.1, C4.1, C5.1, H1.1, H2.1, H3.1, H4.1, J1.B4, J1.B5, J1.B6, J1.SH1, J1.SH2, J1.SH3, J1.SH4, J2.A1, J2.A2, J2.A3, J2.A4, J2.A5, J2.A6, J2.SH1, J2.SH2, J2.SH3, J2.SH4, J3.A1, J3.A2, J3.A3, J3.A4, J3.A5, J3.A6, J3.SH1, J3.SH2, J3.SH3, J3.SH4, J4.A1, J4.A2, J4.A3, J4.A4, J4.A5, J4.A6, J4.SH1, J4.SH2, J4.SH3, J4.SH4
- net RFM_RESET: now also J1.B13
- net at R_BURN1.1, U1.1 (D): now also U1.2 (D), U1.5 (D), U1.6 (D)
- net 4.2V renamed BAT_VOLTAGE
- net BAT_VOLTAGE: now also C2.2, J1.B7, J1.B8, J1.B9, R1.1
- net CLK renamed ANT_SPI2_SCK
- net ANT_SPI2_SCK: now also J1.A4
- net CS renamed ANT_SPI2_NSS
- net ANT_SPI2_NSS: now also J1.A3
- net MISO renamed ANT_SPI2_MISO
- net ANT_SPI2_MISO: now also J1.A2
- net MOSI renamed ANT_SPI2_MOSI
- net ANT_SPI2_MOSI: now also J1.A1
- removed net PMOS_GATE: MOD1.7 (DIO5), MOD1.7_1 (DIO5__1), U1.3 (G)
- new net: R1.2, U1.3 (G)
- new net +3.3V: J1.B1, J1.B2, J1.B3
- new net BURN_WIRE_EN: J1.A5
- new net EXTERNAL_VOLTAGE: C3.2, C4.2, C5.2, J1.B10, J1.B11, J1.B12, J2.B1, J2.B2, J2.B3, J2.B4, J3.B1, J3.B2, J3.B3, J3.B4, J4.B1, J4.B2, J4.B3, J4.B4
- new net I2C1_SCL: J1.A7, J2.B5
- new net I2C1_SDA: J1.A6, J2.B6
- new net I2C2_SCL: J1.A9, J3.B5
- new net I2C2_SDA: J1.A8, J3.B6
- new net I2C3_SCL: J1.A11, J4.B5
- new net I2C3_SDA: J1.A10, J4.B6
- new net I2C4_SCL: J1.A13
- new net I2C4_SDA: J1.A12
- no-connect marks 14 -> 12
Other:
- note added: "Backplane Connection"
- note added: "Burn Wire Circuit"
- note added: "Solar Board Connections"
- note added: "Sun Sensor"
- note added: "To +X"
- note added: "To -X"
- note added: "To -Y"
- note removed: "Burn Wire & Deployment"
- note removed: "Harwin M55 Connector - Interfaces w/ SPI"
- moved on the sheet: R_BURN1, U1

Commit message: Pushing Routing Changes
Parts:
- C2, R1, R_BURN1, U1: now not fitted
Connections:
- net 3.3V is gone; now on net +3.3V: C1.2, MOD1.13 (3.3V), MOD1.13_1 (3.3V__1)
- net BURN_WIRE_EN: now also R1.2, U1.3 (G)
Other:
- note added: "JLC04161H-3313(Finished thickness1.56mm±10%)"
- note added: "Use this stackup as this has trace width at 6.6 mils"

Commit message: Updates due to changes from backplane
Parts:
- C3, C4, C5: value 47uF -> 22uF; footprint Capacitor_SMD:C_1206_3216Metric_Pad1.33x1.80mm_HandSolder -> Capacitor_SMD:C_1210_3225Metric
Changed lines of the file:
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@@
 			)
 		)
-		(property "Value" "47uF"
+		(property "Value" "22uF"
 			(at 147.32 144.7799 0)
 			(show_name no)
@@
 			)
 		)
-		(property "Footprint" "Capacitor_SMD:C_1206_3216Metric_Pad1.33x1.80mm_HandSolder"
+		(property "Footprint" "Capacitor_SMD:C_1210_3225Metric"
 			(at 144.4752 147.32 0)
 			(hide yes)
@@
 			)
 		)
-		(property "Value" "47uF"
+		(property "Value" "22uF"
 			(at 209.55 144.7799 0)
 			(show_name no)
@@
 			)
 		)
-		(property "Footprint" "Capacitor_SMD:C_1206_3216Metric_Pad1.33x1.80mm_HandSolder"
+		(property "Footprint" "Capacitor_SMD:C_1210_3225Metric"
 			(at 206.7052 147.32 0)
 			(hide yes)
@@
 			)
 		)
-		(property "Value" "47uF"
+		(property "Value" "22uF"
 			(at 273.05 144.7799 0)
 			(show_name no)
@@
 			)
 		)
-		(property "Footprint" "Capacitor_SMD:C_1206_3216Metric_Pad1.33x1.80mm_HandSolder"
+		(property "Footprint" "Capacitor_SMD:C_1210_3225Metric"
 			(at 270.2052 147.32 0)
 			(hide yes)
